Commit message: Kodiak extruder model (URDF, visual, collision meshes) added.

File: src/pychoreo_examples/data/models/kuka_kr6_r900/urdf/extrusion_end_effector.urdf (robot description, URDF)
Before this commit: robot extrusion_end_effector, 2 links, 1 joints
Links:
- link eef_base_link: geometry collision mesh filename=../meshes/kodiak_end_effector/collision/kodiak_extruder_col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 scale=.001 .001 .001; visual mesh filename=../meshes/kodiak_end_effector/visual/kodiak_extruder_visual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 scale=.001 .001 .001
Joints:
- joint eef_base_to_tcp: origin xyz=0.150539 0.001052 0.119157 rpy=0.0 1.57079632679 0.0 -> xyz=0.150779 0.008711 0.113987 rpy=0.0 1.57079632679 0.0

File: src/pychoreo_examples/data/models/kuka_kr6_r900/urdf/kuka_kr6_r900_extrusion.urdf (robot description, URDF)
Before this commit: robot kr6_r900_extrusion, 14 links, 13 joints
Links:
- link eef_base_link: geometry collision mesh filename=../meshes/kodiak_end_effector/collision/kodiak_extruder_col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 scale=.001 .001 .001; visual mesh filename=../meshes/kodiak_end_effector/visual/kodiak_extruder_visual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 scale=.001 .001 .001
Joints:
- joint eef_base_to_tcp: origin xyz=0.150539 0.001052 0.119157 rpy=0.0 1.57079632679 0.0 -> xyz=0.150779 0.008711 0.113987 rpy=0.0 1.57079632679 0.0

Commit message: Add preference_cost to SparseLadderGraph and LadderGraph

File: src/pychoreo_examples/data/models/kuka_kr6_r900/urdf/extrusion_end_effector.urdf (robot description, URDF)
Before this commit: robot extrusion_end_effector, 2 links, 1 joints
Links:
- link eef_base_link: geometry collision mesh filename=../meshes/mini_hotend/collision/mini_hotend_collision.stl scale=.001 .001 .001; visual mesh filename=../meshes/mini_hotend/visual/mini_hotend_visual.stl scale=.001 .001 .001
Joints:
- joint eef_base_to_tcp: origin xyz=0.150779 0.008711 0.113987 rpy=0.0 1.57079632679 0.0 -> xyz=0.136569 0.008654 0.109056 rpy=0.0 1.57079632679 0.0

File: src/pychoreo_examples/data/models/kuka_kr6_r900/urdf/kuka_kr6_r900_extrusion.urdf (robot description, URDF)
Before this commit: robot kr6_r900_extrusion, 14 links, 13 joints
Links:
- link eef_base_link: geometry collision mesh filename=../meshes/mini_hotend/collision/mini_hotend_collision.stl scale=.001 .001 .001; visual mesh filename=../meshes/mini_hotend/visual/mini_hotend_visual.stl scale=.001 .001 .001
Joints:
- joint eef_base_to_tcp: origin xyz=0.150779 0.008711 0.113987 rpy=0.0 1.57079632679 0.0 -> xyz=0.136569 0.008654 0.109056 rpy=0.0 1.57079632679 0.0

File: src/pychoreo_examples/data/models/kuka_kr6_r900/urdf/mit_3-412_workspace.urdf (robot description, URDF)
Before this commit: robot mit_3-412_workspace, 9 links, 8 joints
Joints:
- joint workspace_baselink_to_print_table: origin xyz=0.7 0 0.025 rpy=0 0 0 -> xyz=0.7 0 0.024 rpy=0 0 0
