Commit message: extrusion improvements related to real experiments

File: src/pychoreo_examples/data/models/kuka_kr6_r900/urdf/mit_3-412_workspace.urdf (robot description, URDF)
Before this commit: robot mit_3-412_workspace, 8 links, 7 joints
Links:
- added link print_table; collision mesh filename=../meshes/mit_3-412_workspace/collision/print_table.obj scale=.001 .001 .001
Joints:
- added joint workspace_baselink_to_print_table: type fixed, parent workspace_base_link, child print_table, origin xyz=0.7 0 0.025 rpy=0 0 0

Commit message: Klein_bottle_trail, full tip extrusino EE collision model

File: src/pychoreo_examples/data/models/kuka_kr6_r900/urdf/mit_3-412_workspace.urdf (robot description, URDF)
Before this commit: robot mit_3-412_workspace, 9 links, 8 joints
Joints:
- joint workspace_baselink_to_print_table: origin xyz=0.7 0 0.024 rpy=0 0 0 -> xyz=0.7 0 0.022 rpy=0 0 0
